File: EL_IXM233/EL_MX233/EL_MX233.sch (KiCad schematic (older format))
At the start: 1 part

Commit message: add new library
Parts:
- added C1, C10, C2, C4, C6, C7, C8, C9, C? (x25): 100nF, symbol Device:C_Small
- added C3, C5: 10uF/6.3V, symbol Device:C_Small
- added C? (x2): 33pF, symbol Device:C_Small
- added C? (x2): 100uF/16V, symbol Device:CP1_Small
- added C?: 10uF/10V, symbol Device:CP_Small
- added C? (x5): 15pF, symbol Device:C_Small
- added C? (x16): 22uF/6.3V, symbol Device:C_Small
- added C?: NA, symbol Device:C_Small
- added C? (x2): 10pF, symbol Device:C_Small
- added C?: 1uF, symbol Device:C_Small
- added D?: SS14, symbol Device:D_Schottky
- added GND: tp, symbol Connector:TestPoint
- added J?: RJ45_Amphenol_RJMG1BD3B8K1ANR, Connector_RJ:RJ45_Amphenol_RJMG1BD3B8K1ANR, symbol Connector:RJ45_Amphenol_RJMG1BD3B8K1ANR
- added J? (x2): USB_A, symbol Connector:USB_A
- added L? (x2): FB0805/600R/2A, symbol pspice:INDUCTOR
- added L?: INDUCTOR, symbol pspice:INDUCTOR
- added L?: 2.2uH/1.3A, symbol pspice:INDUCTOR
- added R1: 120, symbol Device:R
- added R2, R3: 1K, symbol Device:R
- added R4, R? (x3): 10K, symbol Device:R
- added R?: 12K, symbol Device:R
- added R?: 12.4K, symbol Device:R
- added R?: NA, symbol Device:R
- added R?: 0R, symbol Device:R
- added R?: 1M, symbol Device:R
- added R? (x2): 560R, symbol Device:R
- added R? (x5): 49.9R, symbol Device:R
- added U2: HY5DU121622D, symbol VIETDD:HY5DU121622D
- added U?: LAN9512, symbol VIETDD:LAN9512
- added U?: MIC2026, symbol VIETDD:MIC2026
- added Y?: 25Mhz, symbol Device:Crystal
- added Y?: Crystal, symbol Device:Crystal
- gave numbers to parts that had none: 1
Connections:
- net DCDC_VDDD: now reaches U1.1 (VDD1)
- net DCDC_VDDD: now also U1.94 (DCDC_VDDD), C?.1, C?.1, C?.1
- net VBAT: now reaches U1.100 (DCDC_BATTERY)
- net VBAT: now also U1.103 (BATT), C?.1, C?.1, C?.1
- net at U1.101 (VDD4P2): now also C?.1, C?.1, D?.1 (K)
- net +5V: now reaches U1.102 (VDD5V)
- net +5V: now also C?.1, C?.1, L?.2
- net at U1.105 (VSSA4): now also U1.112 (VSSA1), U1.118 (VSSA2), U1.30 (VSSD1), U1.98 (DCDC_GND), C?.2, C?.2, C?.2, C?.2, C?.2, C?.2, C?.2, C?.2, C?.2, C?.2, C?.2, C?.2, C?.2, C?.2, C?.2, C?.2, C?.2, C?.2, C?.2, C?.2, C?.2, C?.2, C?.2, C?.2, C?.2
- net +2V5: now reaches U1.106 (VDDM/LRADC4)
- net +2V5: now also U1.38 (VDDIO_EMIQ), U1.45 (VDDIO_EM1), U1.53 (VDDIO_EM2), C2.1, C?.1, C?.1, C?.1, C?.1, R3.1, R4.1
- net DCDC_VDDA: now reaches U1.110 (VDDA1)
- net DCDC_VDDA: now also U1.96 (DCDC_VDDA), C?.1, C?.1, C?.1
- net at U1.117 (VAG): now also C?.1
- net at U1.120 (VDDXTAL): now also C?.1
- net XTAL_P: now reaches U1.121 (XTAL_P)
- net XTAL_P: now also C?.1, Y?.2
- net XTAL_N: now reaches U1.122 (XTAL_N)
- net XTAL_N: now also C?.1, Y?.1
- net USB_DM: now reaches U1.123 (USB_DM)
- net USB_DM: now also U?.58 (USBDM0)
- net USB_DP: now reaches U1.124 (USB_DP)
- net USB_DP: now also U?.59 (USBDP0)
- net 3.3VIO: now reaches U1.18 (VDDIO33_1)
- net 3.3VIO: now also U1.92 (VDDIO33_3), U1.95 (DCDC_VDDIO), C?.1, C?.1, C?.1, C?.1
- net at U1.35 (VSSD2): now also C?.2
- net CLK: now reaches U1.36 (EMI_CLK)
- net CLK: now also U1.37 (EMI_CLKN), R1.1, R1.2, U2.45 (CK), U2.46 (#CK)
- net DQS0: now reaches U1.39 (EMI_DQSO)
- net DQS0: now also U2.16 (LDQS)
- net DQS1: now reaches U1.40 (EMI_DQS1)
- net DQS1: now also U2.51 (UDQS)
- net D0: now reaches U1.41 (EMI_D00)
- net D0: now also U2.2 (DQ0)
- net D2: now reaches U1.42 (EMI_D02)
- net D2: now also U2.5 (DQ2)
- net D1: now reaches U1.43 (EMI_D01)
- net D1: now also U2.4 (DQ1)
- net D3: now reaches U1.44 (EMI_D03)
- net D3: now also U2.7 (DQ3)
- net DQM0: now reaches U1.46 (EMI_DQM0)
- net DQM0: now also U2.20 (LDM)
- net D4: now reaches U1.47 (EMI_D04)
- net D4: now also U2.8 (DQ4)
- net D5: now reaches U1.48 (EMI_D05)
- net D5: now also U2.10 (DQ5)
- net D6: now reaches U1.49 (EMI_D06)
- net D6: now also U2.11 (DQ6)
- net D7: now reaches U1.50 (EMI_D07)
- net D7: now also U2.13 (DQ7)
- net D8: now reaches U1.51 (EMI_D08)
- net D8: now also U2.54 (DQ8)
- net D9: now reaches U1.52 (EMI_D09)
- net D9: now also U2.56 (DQ9)
- net D10: now reaches U1.54 (EMI_D10)
- net D10: now also U2.57 (DQ10)
- net D11: now reaches U1.55 (EMI_D11)
- net D11: now also U2.59 (DQ11)
- net DQM1: now reaches U1.56 (EMI_DQM1)
- net DQM1: now also U2.47 (UDM)
- net D12: now reaches U1.57 (EMI_D12)
- net D12: now also U2.60 (DQ12)
- net D13: now reaches U1.58 (EMI_D13)
- net D13: now also U2.62 (DQ13)
- net D15: now reaches U1.59 (EMI_D15)
- net D15: now also U2.65 (DQ15)
- net D14: now reaches U1.60 (EMI_D14)
- net D14: now also U2.63 (DQ14)
- net CASN: now reaches U1.61 (EMI_CASN)
- net CASN: now also U2.22 (#CAS)
- net RASN: now reaches U1.62 (EMI_RASN)
- net RASN: now also U2.23 (#RAS)
- net CS: now reaches U1.63 (EMI_CE0N)
- net CS: now also R4.2, U2.24 (#CS)
- net A12: now reaches U1.64 (EMI_A12)
- net A12: now also U2.42 (A12)
- net A11: now reaches U1.65 (EMI_A11)
- net A11: now also U2.41 (A11)
- net A10: now reaches U1.66 (EMI_A10)
- net A10: now also U2.28 (A10/AP)
- net A9: now reaches U1.67 (EMI_A09)
- net A9: now also U2.40 (A9)
- net A8: now reaches U1.68 (EMI_A08)
- net A8: now also U2.39 (A8)
- net A7: now reaches U1.69 (EMI_A07)
- net A7: now also U2.38 (A7)
- net A6: now reaches U1.70 (EMI_A06)
- net A6: now also U2.37 (A6)
- net A5: now reaches U1.71 (EMI_A05)
- net A5: now also U2.36 (A5)
- net A4: now reaches U1.72 (EMI_A04)
- net A4: now also U2.35 (A4)
- net A3: now reaches U1.73 (EMI_A03)
- net A3: now also U2.32 (A3)
- net A2: now reaches U1.74 (EMI_A02)
- net A2: now also U2.31 (A2)
- net A1: now reaches U1.75 (EMI_A01)
- net A1: now also U2.30 (A1)
- net A0: now reaches U1.76 (EMI_A00)
- net A0: now also U2.29 (A0)
- net WEN: now reaches U1.77 (EMI_WEN)
- net WEN: now also U2.21 (#WE)
- net CKE: now reaches U1.78 (EMI_CKE)
- net CKE: now also U2.44 (CKE)
- net BA0: now reaches U1.79 (EMI_BAO)
- net BA0: now also U2.26 (BA0)
- net BA1: now reaches U1.80 (EMI_BA1)
- net BA1: now also U2.27 (BA1)
- net at U1.93 (VDD3): now also C?.1
- net at U1.97 (DCDC_LN1): now also C?.1, L?.2
- net at U1.99 (DCDC_LP): now also C?.1, L?.1
- new net: C10.2, C3.2, C4.2, C5.2, C6.2, C7.2, C8.2, C9.2, U2.1 (VDD1), U2.15 (VDDQ3), U2.18 (VDD2), U2.3 (VDDQ1), U2.33 (VDD3), U2.55 (VDDQ4), U2.61 (VDDQ5), U2.9 (VDDQ2)
- new net: C10.1, C3.1, C4.1, C5.1, C6.1, C7.1, C8.1, C9.1, U2.12 (VSSQ2), U2.34 (VSS1), U2.48 (VSS2), U2.52 (VSSQ3), U2.58 (VSSQ4), U2.6 (VSSQ1), U2.64 (VSSQ5), U2.66 (VSS3)
- new net: C1.1, C2.2, R2.1, R3.2, U2.49 (VREF)
- new net: J?.2 (D-), U?.1 (USBDM2)
- new net: R?.1, U?.11 (VBUS_DET)
- new net: R?.1, R?.1, R?.1, U?.12 (NRESET)
- new net: C?.1, C?.1, C?.1, U?.15 (VDD18CORE), U?.38 (VDD18CORE)
- new net: J?.3 (D+), U?.2 (USBDP2)
- new net: R?.2, U?.21 (NLNKA_LED/GPIO1)
- new net: R?.2, U?.22 (NSPD_LED/GPIO2)
- new net: J?.2 (D-), U?.3 (USBDM3)
- new net: J?.3 (D+), U?.4 (USBDP3)
- new net: R?.1, U?.41 (AUTOMDIX_EN)
- new net: C?.1, U?.48 (VDD18ETHPLL)
- new net: R?.1, U?.50 (EXRES)
- new net: C?.1, J?.R3 (RD+), R?.2, U?.52 (RXP)
- new net: C?.1, J?.R6 (RD-), R?.2, U?.53 (RXN)
- new net: C?.1, J?.R1 (TD+), R?.2, U?.55 (TXP)
- new net: C?.1, J?.R2 (TD-), R?.2, U?.56 (TXN)
- new net: C?.1, R?.2, U?.60 (XO), Y?.2
- new net: C?.1, R?.1, U?.61 (XI), Y?.1
- new net: C?.1, L?.1, L?.2, U?.62 (VDD18USBPLL)
- new net: R?.1, U?.63 (USBRBIAS)
- new net: J?.L2 (LEDY_K), R?.1
- new net: J?.L3 (LEDG_K), R?.1
- new net: C?.1, J?.R4 (TCT), J?.R5 (RCT), R?.2
- new net: C?.1, L?.1, U?.7 (IN)
- new net 3v3VREG: C?.1, C?.1, C?.1, C?.1, C?.1, J?.L1 (LEDY_A), J?.L4 (LEDG_A), L?.1, R?.2, R?.2, R?.2, U?.19 (VDD33IO), U?.27 (VDD33IO), U?.28 (NTRST), U?.29 (TMS), U?.30 (TDI), U?.32 (TCK), U?.33 (VDD33IO), U?.39 (VDD33IO), U?.40 (TEST3), U?.46 (VDD33IO)
- new net AVCC: C?.2, C?.2, C?.2, C?.2, C?.2, C?.2, C?.2, L?.2, R?.1, R?.1, R?.1, R?.1, R?.1, U?.10 (VDD33A), U?.49 (VDD33A), U?.5 (VDD33A), U?.51 (VDD33A), U?.54 (VDD33A), U?.57 (VDD33A), U?.64 (VDD33A)
- new net GND: C1.2, C?.1, C?.1, C?.1, C?.1, C?.1, C?.1, C?.1, C?.2, C?.2, C?.2, C?.2, C?.2, C?.2, C?.2, C?.2, C?.2, C?.2, C?.2, C?.2, C?.2, C?.2, C?.2, C?.2, C?.2, C?.2, C?.2, C?.2, C?.2, C?.2, D?.2 (A), GND.1, J?.13 (SHIELD), J?.4 (GND), J?.4 (GND), J?.5 (Shield), J?.5 (Shield), J?.R8 (GND), R2.2, R?.2, R?.2, R?.2, U?.34 (TEST2), U?.44 (CLK24_EN), U?.6 (GND), U?.65 (VSS(FLAG))
- new net PIN18/LCD__D17/LAN_RES: R?.2
- new net PRTCTL2: U?.1 (ENA), U?.14 (PRTCTL2), U?.2 (FLAG_A)
- new net PRTCTL3: U?.16 (PRTCTL3), U?.3 (FLAG_B), U?.4 (ENB)
- new net USB_PWR_A: C?.1, J?.1 (VBUS), U?.8 (OUT_A)
- new net USB_PWR_B: C?.1, J?.1 (VBUS), U?.5 (OUT_B)
- no-connect marks 0 -> 7
Other:
- moved on the sheet: U1

Commit message: add new file design
Parts:
- added C? (x2): 1uF, symbol Device:C_Small
- added J?: HEADPHONES, symbol Connector:AudioJack3_Ground
- added J?: AudioJack3_Ground, symbol Connector:AudioJack3_Ground
- added R? (x2): 47K, symbol Device:R
- added R? (x2): 120R, symbol Device:R
- added R? (x2): 10K, symbol Device:R
- added R? (x2): 4.7K, symbol Device:R
- added SW?: RESET, symbol Switch:SW_DIP_x01
- added T1, T2: BC846B, symbol Device:Q_NPN_BCE
Connections:
- net 3.3VIO: now also SW?.1
- net GND: now also C?.2, C?.2, C?.2, C?.2, C?.2, C?.2, C?.2, C?.2, C?.2, C?.2, C?.2, C?.2, C?.2, C?.2, C?.2, C?.2, C?.2, C?.2, C?.2, C?.2, C?.2, C?.2, C?.2, C?.2, C?.2, U1.105 (VSSA4), U1.112 (VSSA1), U1.118 (VSSA2), U1.30 (VSSD1), U1.98 (DCDC_GND), J?.S, R?.1, R?.1, R?.2, T1.3 (E), T2.1 (B), T2.3 (E)
- net XTAL_N: now also T1.2 (C)
- net XTAL_P: now also T2.2 (C)
- net LRADC1: now reaches U1.107 (LRADC1)
- net LRADC0: now reaches U1.108 (LRADC0)
- net at U1.109 (HPR): now also J?.R, R?.1
- net at U1.111 (HP_VGND): now also J?.S, R?.2, R?.2
- net at U1.113 (HPL): now also J?.T, R?.1
- net at U1.114 (LINE1_INR): now also C?.1
- net at U1.115 (LINE1_INL): now also C?.1
- net MIC: now reaches U1.116 (MIC)
- net PSWITCH: now reaches U1.119 (PSWITCH)
- net DEBUG: now reaches U1.89 (DEBUG)
- new net: R?.1, R?.1, T1.1 (B)
- new net: J?.R, R?.2
- new net: J?.T, R?.2
- new net: C?.2, R?.1, R?.2 (x2)
- new net RESET: R?.2, SW?.2
- no-connect marks 7 -> 8
Other:
- note added: "Place T1, T2 as close as possible Q1"
- moved on the sheet: C1, C10, C2, C3, C4, C5, C6, C7, C8, C9, C?, D?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

Commit message: add new file design
Parts:
- added C? (x2): 22uF/6.3V, symbol Device:C_Small
- added D?: LED, symbol Device:LED
- added D?: BAT54C, Package_TO_SOT_SMD:SOT-23, symbol Diode:BAT54C
- added J1, J2: Conn_01x20, symbol Connector_Generic:Conn_01x20
- added J?: Micro_SD_Card, symbol Connector:Micro_SD_Card
- added J?: JTAG, symbol Connector_Generic:Conn_01x08
- added J? (x2): Conn_01x04, symbol Connector_Generic:Conn_01x04
- added J?: Conn_02x04_Top_Bottom, symbol Connector_Generic:Conn_02x04_Top_Bottom
- added L?: INDUCTOR, symbol pspice:INDUCTOR
- added R? (x11): R, symbol Device:R
- added R?: 10K, symbol Device:R
- added R? (x3): 100K, symbol Device:R
- added R?: 4.7k, symbol Device:R
- added R?: 47K, symbol Device:R
- added TP1: TestPoint, symbol Connector:TestPoint
- U1: footprint (none) -> Package_QFP:TQFP-128_14x14mm_P0.4mm
Connections:
- net 3.3VIO: now also J?.1 (Pin_1), J?.2 (Pin_2), J?.3 (Pin_3), J?.4 (Pin_4), L?.1, R?.1, R?.1, R?.1, R?.1, R?.1, R?.2
- net 3v3VREG: now also J1.19 (Pin_19), J?.1 (Pin_1)
- net DEBUG: now also J?.4 (Pin_4), J?.4 (Pin_4)
- net GND: now also C?.2, C?.2, J1.1 (Pin_1), J1.20 (Pin_20), J?.2 (Pin_2), J?.3 (Pin_3), J?.3 (Pin_3), J?.6 (VSS), J?.9 (SHIELD), R?.1, R?.1, R?.1, R?.1, R?.1, R?.2, R?.2
- net VBAT: now also J2.1 (Pin_1)
- net PIN26/LCD_CS: now reaches U1.10 (LCD_CS)
- net PIN26/LCD_CS: now also J1.10 (Pin_10), R?.2
- net PIN22/LCD_EN/I2C_SCL: now reaches U1.11 (LCD_ENABLE/I2C_SCL)
- net PIN22/LCD_EN/I2C_SCL: now also J1.6 (Pin_6)
- net PIN23/LCD_DISP: now reaches U1.12 (LCD_RESET/GPMI_CE3N)
- net PIN23/LCD_DISP: now also J1.7 (Pin_7)
- net PWM0/DUART_RXD: now reaches U1.125 (PWM0/ROTARYA/DUART_RX)
- net PWM0/DUART_RXD: now also J?.2 (Pin_2)
- net PWM1/DUART_TXD: now reaches U1.126 (PWM1/ROTARYB/DUART_TX)
- net PWM1/DUART_TXD: now also D?.2, R?.1
- net AUART1_TXD: now reaches U1.127 (I2C_SCL/GPMI_RDY2/AUART1_TX)
- net AUART1_RXD: now reaches U1.128 (I2C_SDA/GPMI_CE2N/AUART1_RX)
- net PIN24/LCD_WR: now reaches U1.13 (LCD_WR)
- net PIN24/LCD_WR: now also J1.8 (Pin_8)
- net PIN25/LCD_RS: now reaches U1.14 (LCD_RS)
- net PIN25/LCD_RS: now also J1.9 (Pin_9)
- net PIN21/LCD_HYSNC/I2C_SDA: now reaches U1.15 (LCD_HYSNC/I2C_SDA)
- net PIN21/LCD_HYSNC/I2C_SDA: now also J1.5 (Pin_5)
- net PIN20/LCD_VSYNC: now reaches U1.16 (LCD_VSYNC/LCD_BUSY)
- net PIN20/LCD_VSYNC: now also J1.4 (Pin_4)
- net PIN19/LCD_DOTCLK: now reaches U1.17 (LCD_DOTCK/GMPI_RDY3)
- net PIN19/LCD_DOTCLK: now also J1.3 (Pin_3)
- net PIN17/LCD_D16: now reaches U1.19 (GPMI_CLE/LCD_D16)
- net PIN17/LCD_D16: now also J2.2 (Pin_2)
- net PIN1/LCD_D00: now reaches U1.2 (LCD_DOO)
- net PIN1/LCD_D00: now also J2.18 (Pin_18), R?.1, R?.2
- net PIN18/LCD_D17/LAN_RES: now reaches U1.20 (GPMI_ALE/LCD_D17)
- net PIN18/LCD_D17/LAN_RES: now also J1.2 (Pin_2)
- net SSP2_MOSI: now reaches U1.21 (GPMI_RDY1/SSP2_CMD)
- net PIN9/LCD_D08/SSP2_MISO: now reaches U1.22 (GPMI_D00/LCD_D08/SSP2_DATA0)
- net PIN9/LCD_D08/SSP2_MISO: now also J2.10 (Pin_10)
- net PIN10/LCD_D09: now reaches U1.23 (GPMI_D01/LCD_D09/SSP2_DATA1)
- net PIN10/LCD_D09: now also J2.9 (Pin_9)
- net PIN11/LCD_D10: now reaches U1.24 (GPMI_D02/LCD_D10/SSP2_DATA2)
- net PIN11/LCD_D10: now also J2.8 (Pin_8)
- net PIN12/LCD_D11/UEXT_CS: now reaches U1.25 (GPMI_D03/LCD_D11/SSP2_DATA3)
- net PIN12/LCD_D11/UEXT_CS: now also J2.7 (Pin_7)
- net PIN14/LCD_D13: now reaches U1.26 (GPMI_D05/LCD_D13/SSP2_DATA5)
- net PIN14/LCD_D13: now also J2.5 (Pin_5)
- net PIN13/LCD_D12: now reaches U1.27 (GPMI_D04/LCD_D12/SSP2_DATA4)
- net PIN13/LCD_D12: now also J2.6 (Pin_6)
- net PIN16/LCD_D15: now reaches U1.28 (GPMI_D07/LCD_D15/SSP2_DATA7)
- net PIN16/LCD_D15: now also J2.3 (Pin_3)
- net PIN15/LCD_D14: now reaches U1.29 (GPMI_D06/LCD_D14/SSP2_DATA6)
- net PIN15/LCD_D14: now also J2.4 (Pin_4)
- net PIN2/LCD_D01: now reaches U1.3 (LCD_DO1)
- net PIN2/LCD_D01: now also J2.17 (Pin_17), R?.1, R?.2
- net PIN28/SOFT_SDA: now reaches U1.31 (GPMI_RDN)
- net PIN28/SOFT_SDA: now also J1.12 (Pin_12)
- net TEST_PAD: now reaches U1.32 (GPMI_RDY0/SSP2_DETECT)
- net TEST_PAD: now also TP1.1
- net SSP2_SCK: now reaches U1.33 (GPMI_WRN/SSP2_SCK)
- net PIN29/SOFT_SCL: now reaches U1.34 (GPMI_WPN)
- net PIN29/SOFT_SCL: now also J1.13 (Pin_13)
- net PIN3/LCD_D02: now reaches U1.4 (LCD_DO2)
- net PIN3/LCD_D02: now also J2.16 (Pin_16), R?.1, R?.2
- net PIN4/LCD_D03: now reaches U1.5 (LCD_DO3)
- net PIN4/LCD_D03: now also J2.15 (Pin_15), R?.1, R?.2
- net PIN5/LCD_D04: now reaches U1.6 (LCD_DO4)
- net PIN5/LCD_D04: now also J2.14 (Pin_14)
- net PIN6/LCD_D05: now reaches U1.7 (LCD_DO5)
- net PIN6/LCD_D05: now also J2.13 (Pin_13), R?.2
- net PIN7/LCD_D06: now reaches U1.8 (LCD_DO6)
- net PIN7/LCD_D06: now also J2.12 (Pin_12)
- net PIN30: now reaches U1.81 (GPMI_1N)
- net PIN30: now also J1.14 (Pin_14)
- net PIN31: now reaches U1.82 (GPMI_0N)
- net PIN31: now also J1.15 (Pin_15)
- net SSP1_CMD: now reaches U1.83 (SSP1_CMD/SPI1_MOSI/JTAG_TDO)
- net SSP1_CMD: now also J?.3 (CMD), J?.6 (Pin_6), R?.2
- net SSP1_DATA0: now reaches U1.84 (SSP1_DATA0/SPI1_MISO/JTAG_TDI)
- net SSP1_DATA0: now also J?.2 (Pin_2), J?.7 (DAT0), R?.2
- net SSP1_DATA1: now reaches U1.85 (SSP1_DATA1/I2C_SCL/JTAG_TCLK)
- net SSP1_DATA1: now also J?.1 (Pin_1), J?.8 (DAT1), R?.2
- net SSP1_DATA2: now reaches U1.86 (SSP1_DATA2/I2C_SDA/JTAG_RCLK)
- net SSP1_DATA2: now also J?.1 (DAT2), J?.8 (Pin_8), R?.2
- net SSP1_DATA3: now reaches U1.87 (SSP1_DATA3/SPI1_SS/JTAG_TMS)
- net SSP1_DATA3: now also J?.2 (DAT3/CD), J?.7 (Pin_7), R?.1
- net LED1: now reaches U1.88 (SSP1_DETECT/GPMI_CE3N/USB_ID)
- net LED1: now also D?.2 (A)
- net PIN8/LCD_D07: now reaches U1.9 (LCD_DO7)
- net PIN8/LCD_D07: now also J2.11 (Pin_11)
- net SSP1_SCK: now reaches U1.90 (SSP1_SCK/SPI1_SCK/JTAG_TRST)
- net SSP1_SCK: now also J?.4 (Pin_4), J?.5 (CLK)
- net PIN27/PWM2: now reaches U1.91 (PWM2/GPMI_RDY3)
- net PIN27/PWM2: now also J1.11 (Pin_11)
- net LRADC0 renamed PIN33/LRADC0
- net PIN33/LRADC0: now also J1.17 (Pin_17)
- net LRADC1 renamed PIN32/LRADC1
- net PIN32/LRADC1: now also J1.16 (Pin_16)
- net MIC renamed PIN34/MIC
- net PIN34/MIC: now also J1.18 (Pin_18)
- new net: D?.1 (K), R?.1
- new net: D?.3, J?.1 (Pin_1)
- new net: J?.5 (Pin_5), R?.2
- new net: J?.6 (Pin_6), R?.2
- new net: J?.7 (Pin_7), R?.2
- new net: J?.8 (Pin_8), R?.2
- new net +5VEXT: J2.19 (Pin_19)
- new net SD_VCC: C?.1, C?.1, J?.4 (VDD), J?.5 (Pin_5), L?.2
- new net SJTAG_PSW: J?.3 (Pin_3)
- new net VIN: J2.20 (Pin_20)
